File: schematic/KiCad/Solar_charger3a.sch (KiCad schematic (older format))
At the start: 59 parts, among them J1 SOLAR INPUT, J2 Load Terminal, J3 BATTERY, J4 ESP01 connector, J5 LED Conn, J6 LCD Conn, Q1 IRFZ44N, Q2 IRFZ44N, Q3 IRFZ44N, Q4 IRFZ44N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

Commit message: minor updates
Connections:
- wire segments 107 -> 140
Other:
- moved on the sheet: C10, C3, J1, R1, R2, R24
